Commit message: First bits of the assembly manager

File: flat_bot_support/urdf/flat_bot_macro.xacro (robot description, xacro)
@@ -175,9 +175,9 @@
     </joint>
     <joint name="${prefix}latch_a_joint" type="revolute">
-      <origin xyz="0.0565 0.021472 0.038" rpy="0 0 ${-pi/4}"/>
+      <origin xyz="0.043857 0.018472 0.038" rpy="0 0 ${(3*pi)/4}"/>
       <parent link="${prefix}sirom_a_link"/>
       <child link="${prefix}sirom_a_latch"/>
       <axis xyz="0 0 1"/>
-      <limit lower="-0.2" upper="${pi}" effort="100" velocity="${(2*pi)+0.2}"/>
+      <limit lower="${-pi-0.2}" upper="${0.2}" effort="100" velocity="${(2*pi)}"/>
     </joint>
     <joint name="${prefix}latch_b_joint" type="revolute">
@@ -186,5 +186,5 @@
       <child link="${prefix}sirom_b_latch"/>
       <axis xyz="0 0 1"/>
-      <limit lower="-0.2" upper="${pi}" effort="100" velocity="${(2*pi)+0.2}"/>
+      <limit lower="-0.2" upper="${pi+0.2}" effort="100" velocity="${(2*pi)}"/>
     </joint>
     <!-- transform from the standard SIROM frame to the sirom_b link -->

File: flat_bot_support/urdf/passive_sirom_macro.xacro (robot description, xacro)
@@ -4,4 +4,26 @@
   <static>true</static>
     <!-- links: main serial chain -->
+    <link name="${prefix}track_link">
+      <visual>
+        <origin xyz="0 0 0" rpy="0 0 0"/>
+        <geometry>
+          <mesh filename="package://flat_bot_support/meshes/visual/four_sirom_track.stl" />
+        </geometry>
+      </visual>
+      <collision>
+        <origin xyz="0 0 0" rpy="0 0 0"/>
+        <geometry>
+          <mesh filename="package://flat_bot_support/meshes/visual/four_sirom_track.stl" />
+        </geometry>
+      </collision>
+      <inertial>
+        <mass value="5.523" />
+        <origin xyz="0.080698 -0.600207 0.025679" rpy="0 -0.0211184839491314 0" />
+        <inertia
+          ixx="0.822090658" ixy="0.0" ixz="0.0"
+          iyy="0.004754978" iyz="0.0"
+          izz="0.824462923" />
+      </inertial>
+    </link>
     <link name="${prefix}sirom_a_link">
       <visual>
@@ -26,4 +48,9 @@
       </inertial>
     </link>
+    <joint name="temp_joint" type="fixed">
+      <origin xyz="-0.20 0 0" rpy="0 0 0"/>
+      <parent link="${prefix}track_link"/>
+      <child link="${prefix}sirom_a_link"/>
+    </joint>
   </xacro:macro>
 </robot>

Commit message: added robot base link module to manager and first assembly sim demo

File: flat_bot_support/urdf/flat_bot_macro.xacro (robot description, xacro)
@@ -9,8 +9,8 @@
     </gazebo>
     <!-- placeholder links to define the connector coordinate frames of each end effector -->
-    <link name="${prefix}sirom_a_origin">
+    <!--link name="${prefix}sirom_a_origin">
     </link>
     <link name="${prefix}sirom_b_origin">
-    </link>
+    </link-->
     <!-- links: main serial chain -->
     <link name="${prefix}sirom_a_link">
@@ -147,9 +147,9 @@
     </link>
     <!-- transforms from the standard SIROM frame to the sirom_a link -->
-    <joint name="${prefix}sirom_a_origin-link" type="fixed">
+    <!--joint name="${prefix}sirom_a_origin-link" type="fixed">
       <origin xyz="0 0 0" rpy="0 0 ${pi}"/>
       <parent link="${prefix}sirom_a_origin"/>
       <child link="${prefix}sirom_a_link"/>
-    </joint>
+    </joint-->
     <!-- joints: main serial chain -->
     <joint name="${prefix}wrist_a_joint" type="revolute">
@@ -189,9 +189,9 @@
     </joint>
     <!-- transform from the standard SIROM frame to the sirom_b link -->
-    <joint name="${prefix}sirom_b_link-origin" type="fixed">
+    <!--joint name="${prefix}sirom_b_link-origin" type="fixed">
       <origin xyz="0.0785 -0.0213 0" rpy="0 0 0" />
       <parent link="${prefix}sirom_b_link" />
       <child link="${prefix}sirom_b_origin" />
-    </joint>
+    </joint-->
     <!-- ================= Arm Joint Transmissions ==================== -->
     <transmission name="wrist_a_trans">
